File: PCB/printplaat2/pcb_PoAB/pcb_PoAB.kicad_sch (KiCad schematic)
At the start: 34 parts, among them J1 battertij, J10 GPS, J2 lichtmeter1, J3 lichtmeter2, J4 lichtmeter3, J5 lichtmeter4, J6 lamp1, J7 lamp2, J8 lamp3, J9 spannigsmeter, U1 L7805CV, U2 AQY211EHAZ, U3 AQY211EHAZ, U4 AQY211EHAZ, U5 ACS712ELCTR-05B-T, U6 ACS712ELCTR-05B-T, U7 ACS712ELCTR-05B-T, U8 ADS1115, U9 ARDUINO_MKR_WAN_1310

Commit message: pcb baseplate aangepast
Parts:
- renumbered U1 to 5V_Reg1, U8 to ADC_I²C1, U5 to A_meter1, U6 to A_meter2, U7 to A_meter3, J1 to Bat1, J10 to GPS1, J2 to LuxMeter1, J3 to LuxMeter2, J4 to LuxMeter3, J5 to LuxMeter4, U2 to Mos1, U3 to Mos2, U4 to Mos3, J9 to V_Meter1, J6 to lamp1, J7 to lamp2, J8 to lamp3
Connections:
- net +3.3V: now also V_Meter1.1 (Pin_1)
- net 5V_bord: no longer V_Meter1.1 (Pin_1)
- net RX: now also U9.J5_8 (PB23/D13/RX(SC5)); no longer U9.J5_9 (PB22/D14/TX(SC5))
- net TX: now also U9.J5_9 (PB22/D14/TX(SC5)); no longer U9.J5_8 (PB23/D13/RX(SC5))
- no-connect marks 13 -> 14

Commit message: pcb zip gemaakt
Other:
- title: (none) -> POAB_Baseplate
Changed lines of the file:
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@@
 (kicad_sch (version 20211123) (generator eeschema)
   (paper "A4")
+  (title_block
+    (title "POAB_Baseplate")
+    (date "2023-05-16")
+    (rev "2.0")
+    (comment 2 "Quinten Moons & Kevin Lahey")
+  )
   (junction (at 101.092 144.78) (diameter 0) (color 0 0 0 0)
   )
