File: PCB/printplaat2/pcb_PoAB/lichtsensor/lichtsensor.kicad_sch (KiCad schematic)
At the start: 3 parts, among them J1 Conn_01x03_Male, Q1 TEMT6000X01

Commit message: pcb zip gemaakt
Parts:
- added H1, H2, H3, H4: MountingHole_Pad, Connector_PinSocket_1.27mm:PinSocket_1x01_P1.27mm_Vertical, symbol Mechanical:MountingHole_Pad
Connections:
- net GND: now also H1.1, H2.1, H3.1, H4.1
Other:
- moved on the sheet: J1
Changed lines of the file:
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@@
 (kicad_sch (version 20211123) (generator eeschema)
   (paper "A4")
+  (junction (at 195.58 80.01) (diameter 0) (color 0 0 0 0)
+  )
+  (junction (at 195.58 91.44) (diameter 0) (color 0 0 0 0)
+  )
   (junction (at 121.92 78.74) (diameter 0) (color 0 0 0 0)
   )
+  (junction (at 195.58 68.58) (diameter 0) (color 0 0 0 0)
+  )
+  (wire (pts (xy 195.58 57.15) (xy 195.58 68.58))
+    (stroke (width 0) (type default) (color 0 0 0 0))
+  )
   (wire (pts (xy 121.92 59.69) (xy 121.92 64.77))
     (stroke (width 0) (type default) (color 0 0 0 0))
@@
     (stroke (width 0) (type default) (color 0 0 0 0))
   )
-  (wire (pts (xy 162.56 63.5) (xy 162.56 68.58))
+  (wire (pts (xy 187.96 91.44) (xy 195.58 91.44))
+    (stroke (width 0) (type default) (color 0 0 0 0))
+  )
+  (wire (pts (xy 158.75 63.5) (xy 158.75 68.58))
     (stroke (width 0) (type default) (color 0 0 0 0))
   )
@@
     (stroke (width 0) (type default) (color 0 0 0 0))
   )
-  (wire (pts (xy 152.4 63.5) (xy 152.4 67.31))
-    (stroke (width 0) (type default) (color 0 0 0 0))
-  )
-  (wire (pts (xy 157.48 67.31) (xy 157.48 63.5))
-    (stroke (width 0) (type default) (color 0 0 0 0))
-  )
-  (wire (pts (xy 160.02 63.5) (xy 160.02 71.12))
-    (stroke (width 0) (type default) (color 0 0 0 0))
-  )
-  (wire (pts (xy 152.4 67.31) (xy 157.48 67.31))
+  (wire (pts (xy 187.96 68.58) (xy 195.58 68.58))
+    (stroke (width 0) (type default) (color 0 0 0 0))
+  )
+  (wire (pts (xy 148.59 63.5) (xy 148.59 67.31))
+    (stroke (width 0) (type default) (color 0 0 0 0))
+  )
+  (wire (pts (xy 153.67 67.31) (xy 153.67 63.5))
+    (stroke (width 0) (type default) (color 0 0 0 0))
+  )
+  (wire (pts (xy 195.58 68.58) (xy 195.58 80.01))
+    (stroke (width 0) (type default) (color 0 0 0 0))
+  )
+  (wire (pts (xy 187.96 80.01) (xy 195.58 80.01))
+    (stroke (width 0) (type default) (color 0 0 0 0))
+  )
+  (wire (pts (xy 156.21 63.5) (xy 156.21 71.12))
+    (stroke (width 0) (type default) (color 0 0 0 0))
+  )
+  (wire (pts (xy 195.58 80.01) (xy 195.58 91.44))
+    (stroke (width 0) (type default) (color 0 0 0 0))
+  )
+  (wire (pts (xy 187.96 57.15) (xy 195.58 57.15))
+    (stroke (width 0) (type default) (color 0 0 0 0))
+  )
+  (wire (pts (xy 148.59 67.31) (xy 153.67 67.31))
+    (stroke (width 0) (type default) (color 0 0 0 0))
+  )
+  (wire (pts (xy 195.58 91.44) (xy 195.58 99.06))
     (stroke (width 0) (type default) (color 0 0 0 0))
   )
@@
     (effects (font (size 1.27 1.27)) (justify right bottom))
   )
-  (label "output" (at 160.02 71.12 180)
+  (label "output" (at 156.21 71.12 180)
     (effects (font (size 1.27 1.27)) (justify right bottom))
   )
-  (symbol (lib_id "power:VCC") (at 152.4 63.5 0) (unit 1)
-    (in_bom yes) (on_board yes) (fields_autoplaced)
-    (property "Reference" "#PWR03" (id 0) (at 152.4 67.31 0)
-      (effects (font (size 1.27 1.27)) hide)
-    )
-    (property "Value" "VCC" (id 1) (at 152.4 58.42 0))
-    (property "Footprint" "" (id 2) (at 152.4 63.5 0)
-      (effects (font (size 1.27 1.27)) hide)
-    )
-    (property "Datasheet" "" (id 3) (at 152.4 63.5 0)
+  (symbol (lib_id "power:VCC") (at 148.59 63.5 0) (unit 1)
+    (in_bom yes) (on_board yes) (fields_autoplaced)
+    (property "Reference" "#PWR03" (id 0) (at 148.59 67.31 0)
+      (effects (font (size 1.27 1.27)) hide)
+    )
+    (property "Value" "VCC" (id 1) (at 148.59 58.42 0))
+    (property "Footprint" "" (id 2) (at 148.59 63.5 0)
+      (effects (font (size 1.27 1.27)) hide)
+    )
+    (property "Datasheet" "" (id 3) (at 148.59 63.5 0)
       (effects (font (size 1.27 1.27)) hide)
     )
@@
     (pin "1")
   )
+  (symbol (lib_id "Mechanical:MountingHole_Pad") (at 185.42 57.15 90) (unit 1)
+    (in_bom yes) (on_board yes) (fields_autoplaced)
+    (property "Reference" "H1" (id 0) (at 184.15 49.53 90))
+    (property "Value" "MountingHole_Pad" (id 1) (at 184.15 52.07 90))
+    (property "Footprint" "Connector_PinSocket_1.27mm:PinSocket_1x01_P1.27mm_Vertical" (id 2) (at 185.42 57.15 0)
+      (effects (font (size 1.27 1.27)) hide)
+    )
+    (property "Datasheet" "~" (id 3) (at 185.42 57.15 0)
+      (effects (font (size 1.27 1.27)) hide)
+    )
+    (pin "1")
+  )
   (symbol (lib_id "TEMT6000X01:TEMT6000X01") (at 119.38 69.85 0) (unit 1)
     (in_bom yes) (on_board yes) (fields_autoplaced)
@@
     (pin "3")
   )
+  (symbol (lib_id "power:GND") (at 195.58 99.06 0) (unit 1)
+    (in_bom yes) (on_board yes)
+    (property "Reference" "#PWR05" (id 0) (at 195.58 105.41 0)
+      (effects (font (size 1.27 1.27)) hide)
+    )
+    (property "Value" "GND" (id 1) (at 195.58 104.14 0))
+    (property "Footprint" "" (id 2) (at 195.58 99.06 0)
+      (effects (font (size 1.27 1.27)) hide)
+    )
+    (property "Datasheet" "" (id 3) (at 195.58 99.06 0)
+      (effects (font (size 1.27 1.27)) hide)
+    )
+    (pin "1")
+  )
+  (symbol (lib_id "Mechanical:MountingHole_Pad") (at 185.42 91.44 90) (unit 1)
+    (in_bom yes) (on_board yes) (fields_autoplaced)
+    (property "Reference" "H4" (id 0) (at 184.15 83.82 90))
+    (property "Value" "MountingHole_Pad" (id 1) (at 184.15 86.36 90))
+    (property "Footprint" "Connector_PinSocket_1.27mm:PinSocket_1x01_P1.27mm_Vertical" (id 2) (at 185.42 91.44 0)
+      (effects (font (size 1.27 1.27)) hide)
+    )
+    (property "Datasheet" "~" (id 3) (at 185.42 91.44 0)
+      (effects (font (size 1.27 1.27)) hide)
+    )
+    (pin "1")
+  )
+  (symbol (lib_id "Mechanical:MountingHole_Pad") (at 185.42 80.01 90) (unit 1)
+    (in_bom yes) (on_board yes) (fields_autoplaced)
+    (property "Reference" "H3" (id 0) (at 184.15 72.39 90))
+    (property "Value" "MountingHole_Pad" (id 1) (at 184.15 74.93 90))
+    (property "Footprint" "Connector_PinSocket_1.27mm:PinSocket_1x01_P1.27mm_Vertical" (id 2) (at 185.42 80.01 0)
+      (effects (font (size 1.27 1.27)) hide)
+    )
+    (property "Datasheet" "~" (id 3) (at 185.42 80.01 0)
+      (effects (font (size 1.27 1.27)) hide)
+    )
+    (pin "1")
+  )
   (symbol (lib_id "Device:R") (at 121.92 85.09 0) (unit 1)
     (in_bom yes) (on_board yes) (fields_autoplaced)
@@
     (pin "2")
   )
-  (symbol (lib_id "Connector:Conn_01x03_Male") (at 160.02 58.42 270) (unit 1)
-    (in_bom yes) (on_board yes) (fields_autoplaced)
-    (property "Reference" "J1" (id 0) (at 160.02 53.34 90))
-    (property "Value" "Conn_01x03_Male" (id 1) (at 160.02 55.88 90))
-    (property "Footprint" "Connector_PinSocket_2.54mm:PinSocket_1x03_P2.54mm_Vertical" (id 2) (at 160.02 58.42 0)
-      (effects (font (size 1.27 1.27)) hide)
-    )
-    (property "Datasheet" "~" (id 3) (at 160.02 58.42 0)
+  (symbol (lib_id "Mechanical:MountingHole_Pad") (at 185.42 68.58 90) (unit 1)
+    (in_bom yes) (on_board yes) (fields_autoplaced)
+    (property "Reference" "H2" (id 0) (at 184.15 60.96 90))
+    (property "Value" "MountingHole_Pad" (id 1) (at 184.15 63.5 90))
+    (property "Footprint" "Connector_PinSocket_1.27mm:PinSocket_1x01_P1.27mm_Vertical" (id 2) (at 185.42 68.58 0)
+      (effects (font (size 1.27 1.27)) hide)
+    )
+    (property "Datasheet" "~" (id 3) (at 185.42 68.58 0)
+      (effects (font (size 1.27 1.27)) hide)
+    )
+    (pin "1")
+  )
+  (symbol (lib_id "Connector:Conn_01x03_Male") (at 156.21 58.42 270) (unit 1)
+    (in_bom yes) (on_board yes) (fields_autoplaced)
+    (property "Reference" "J1" (id 0) (at 156.21 53.34 90))
+    (property "Value" "Conn_01x03_Male" (id 1) (at 156.21 55.88 90))
+    (property "Footprint" "Connector_PinSocket_2.54mm:PinSocket_1x03_P2.54mm_Vertical" (id 2) (at 156.21 58.42 0)
+      (effects (font (size 1.27 1.27)) hide)
+    )
+    (property "Datasheet" "~" (id 3) (at 156.21 58.42 0)
       (effects (font (size 1.27 1.27)) hide)
     )
@@
     (pin "1")
   )
-  (symbol (lib_id "power:GND") (at 162.56 68.58 0) (unit 1)
+  (symbol (lib_id "power:GND") (at 158.75 68.58 0) (unit 1)
     (in_bom yes) (on_board yes)
-    (property "Reference" "#PWR04" (id 0) (at 162.56 74.93 0)
-      (effects (font (size 1.27 1.27)) hide)
-    )
-    (property "Value" "GND" (id 1) (at 162.56 73.66 0))
-    (property "Footprint" "" (id 2) (at 162.56 68.58 0)
-      (effects (font (size 1.27 1.27)) hide)
-    )
-    (property "Datasheet" "" (id 3) (at 162.56 68.58 0)
+    (property "Reference" "#PWR04" (id 0) (at 158.75 74.93 0)
+      (effects (font (size 1.27 1.27)) hide)
+    )
+    (property "Value" "GND" (id 1) (at 158.75 73.66 0))
+    (property "Footprint" "" (id 2) (at 158.75 68.58 0)
+      (effects (font (size 1.27 1.27)) hide)
+    )
+    (property "Datasheet" "" (id 3) (at 158.75 68.58 0)
       (effects (font (size 1.27 1.27)) hide)
     )
@@
       (reference "#PWR04") (unit 1) (value "GND") (footprint "")
     )
+    (path "/32d4d97c-4648-4b16-9a25-e0f6c6b14c2b"
+      (reference "#PWR05") (unit 1) (value "GND") (footprint "")
+    )
+    (path "/2d4765ff-cb61-478a-82dd-c4469ff0841b"
+      (reference "H1") (unit 1) (value "MountingHole_Pad") (footprint "Connector_PinSocket_1.27mm:PinSocket_1x01_P1.27mm_Vertical")
+    )
+    (path "/97f3e72c-5c8c-4cc3-b86e-4ea40df2a26e"
+      (reference "H2") (unit 1) (value "MountingHole_Pad") (footprint "Connector_PinSocket_1.27mm:PinSocket_1x01_P1.27mm_Vertical")
+    )
+    (path "/5e47ce77-07ac-4dd3-b666-284b3cff64ec"
+      (reference "H3") (unit 1) (value "MountingHole_Pad") (footprint "Connector_PinSocket_1.27mm:PinSocket_1x01_P1.27mm_Vertical")
+    )
+    (path "/50e4ac08-1c5c-4389-a1a0-88496fddc8ff"
+      (reference "H4") (unit 1) (value "MountingHole_Pad") (footprint "Connector_PinSocket_1.27mm:PinSocket_1x01_P1.27mm_Vertical")
+    )
     (path "/a6409935-bd2f-4c98-bc2d-1beb0b433ae4"
