File: PCB/Moons_Quinten_PCB/printplaat2/pcb_PoAB/lichtsensor/lichtsensor.kicad_sch (KiCad schematic)
At the start: 7 parts, among them J1 Conn_01x03_Male, Q1 TEMT6000X01

Commit message: pcb lichtsensor aangepast
Parts:
- H1, H2, H3, H4: footprint Connector_PinSocket_1.27mm:PinSocket_1x01_P1.27mm_Vertical -> MountingHole:MountingHole_2.1mm
Changed lines of the file:
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@@
     (property "Reference" "H1" (id 0) (at 184.15 49.53 90))
     (property "Value" "MountingHole_Pad" (id 1) (at 184.15 52.07 90))
-    (property "Footprint" "Connector_PinSocket_1.27mm:PinSocket_1x01_P1.27mm_Vertical" (id 2) (at 185.42 57.15 0)
+    (property "Footprint" "MountingHole:MountingHole_2.1mm" (id 2) (at 185.42 57.15 0)
       (effects (font (size 1.27 1.27)) hide)
     )
@@
     (property "Reference" "H4" (id 0) (at 184.15 83.82 90))
     (property "Value" "MountingHole_Pad" (id 1) (at 184.15 86.36 90))
-    (property "Footprint" "Connector_PinSocket_1.27mm:PinSocket_1x01_P1.27mm_Vertical" (id 2) (at 185.42 91.44 0)
+    (property "Footprint" "MountingHole:MountingHole_2.1mm" (id 2) (at 185.42 91.44 0)
       (effects (font (size 1.27 1.27)) hide)
     )
@@
     (property "Reference" "H3" (id 0) (at 184.15 72.39 90))
     (property "Value" "MountingHole_Pad" (id 1) (at 184.15 74.93 90))
-    (property "Footprint" "Connector_PinSocket_1.27mm:PinSocket_1x01_P1.27mm_Vertical" (id 2) (at 185.42 80.01 0)
+    (property "Footprint" "MountingHole:MountingHole_2.1mm" (id 2) (at 185.42 80.01 0)
       (effects (font (size 1.27 1.27)) hide)
     )
@@
     (property "Reference" "H2" (id 0) (at 184.15 60.96 90))
     (property "Value" "MountingHole_Pad" (id 1) (at 184.15 63.5 90))
-    (property "Footprint" "Connector_PinSocket_1.27mm:PinSocket_1x01_P1.27mm_Vertical" (id 2) (at 185.42 68.58 0)
+    (property "Footprint" "MountingHole:MountingHole_2.1mm" (id 2) (at 185.42 68.58 0)
       (effects (font (size 1.27 1.27)) hide)
     )
@@
     )
     (path "/2d4765ff-cb61-478a-82dd-c4469ff0841b"
-      (reference "H1") (unit 1) (value "MountingHole_Pad") (footprint "Connector_PinSocket_1.27mm:PinSocket_1x01_P1.27mm_Vertical")
+      (reference "H1") (unit 1) (value "MountingHole_Pad") (footprint "MountingHole:MountingHole_2.1mm")
     )
     (path "/97f3e72c-5c8c-4cc3-b86e-4ea40df2a26e"
-      (reference "H2") (unit 1) (value "MountingHole_Pad") (footprint "Connector_PinSocket_1.27mm:PinSocket_1x01_P1.27mm_Vertical")
+      (reference "H2") (unit 1) (value "MountingHole_Pad") (footprint "MountingHole:MountingHole_2.1mm")
     )
     (path "/5e47ce77-07ac-4dd3-b666-284b3cff64ec"
-      (reference "H3") (unit 1) (value "MountingHole_Pad") (footprint "Connector_PinSocket_1.27mm:PinSocket_1x01_P1.27mm_Vertical")
+      (reference "H3") (unit 1) (value "MountingHole_Pad") (footprint "MountingHole:MountingHole_2.1mm")
     )
     (path "/50e4ac08-1c5c-4389-a1a0-88496fddc8ff"
-      (reference "H4") (unit 1) (value "MountingHole_Pad") (footprint "Connector_PinSocket_1.27mm:PinSocket_1x01_P1.27mm_Vertical")
+      (reference "H4") (unit 1) (value "MountingHole_Pad") (footprint "MountingHole:MountingHole_2.1mm")
     )
     (path "/a6409935-bd2f-4c98-bc2d-1beb0b433ae4"
